Commit message: namespace tweaks

File: urdf/cora_p3d.xacro (robot description, xacro)
@@ -12,8 +12,11 @@
   <xacro:arg name="namespace" default="cora"/>
   <xacro:property name="namespace" value="$(arg namespace)" scope="global" />
+  <!-- Thrusters mess this up - so this is hack - TODO Fix! -->
+  <xacro:arg name="root_namespace" default=""/>
+  <xacro:property name="root_namespace" value="$(arg root_namespace)" scope="global" />
   <!-- Thrusters -->
   <xacro:arg name="thruster_namespace" default="thrusters/"/>
   <xacro:property name="thruster_namespace" value="$(arg thruster_namespace)" scope="global" />
-  <xacro:include filename="$(find cora_description)/urdf/thrusters.xacro" />
+  <xacro:include filename="$(find mrc_examples)/urdf/thrusters.xacro" />
   <!-- Decide if we lock the robot to the world -->
   <xacro:if value="$(arg locked)">

Commit message: This looks like it fixed the issue

File: urdf/cora_p3d.xacro (robot description, xacro)
@@ -12,11 +12,8 @@
   <xacro:arg name="namespace" default="cora"/>
   <xacro:property name="namespace" value="$(arg namespace)" scope="global" />
-  <!-- Thrusters mess this up - so this is hack - TODO Fix! -->
-  <xacro:arg name="root_namespace" default=""/>
-  <xacro:property name="root_namespace" value="$(arg root_namespace)" scope="global" />
   <!-- Thrusters -->
   <xacro:arg name="thruster_namespace" default="thrusters/"/>
   <xacro:property name="thruster_namespace" value="$(arg thruster_namespace)" scope="global" />
-  <xacro:include filename="$(find mrc_examples)/urdf/thrusters.xacro" />
+  <xacro:include filename="$(find cora_description)/urdf/thrusters.xacro" />
   <!-- Decide if we lock the robot to the world -->
   <xacro:if value="$(arg locked)">
@@ -24,5 +21,5 @@
       <link name="cora_external_link"/>
       <joint name="cora_external_pivot_joint" type="universal">
-        <parent>cora::base_link</parent>
+        <parent>cora::cora/base_link</parent>
         <child>cora_external_link</child>
         <axis>
@@ -53,14 +50,16 @@
   <xacro:property name="sensor_namespace" value="$(arg sensor_namespace)" scope="global" />
   <xacro:property name="pinger_namespace" value="$(arg pinger_namespace)" scope="global" />
-  <xacro:wamv_camera name="front_left_camera"  x="-0.61" y="0.2"  z="4.7" post_z_from="4.6" P="${radians(15)}" />
-  <xacro:wamv_camera name="front_right_camera" x="-0.61" y="-0.2" z="4.7" post_z_from="4.6" P="${radians(15)}" />
-  <xacro:lidar name="front_lidar" type="16_beam" x="-0.595" z="5" P="${radians(8)}" post_z_from="4.6"/>
-  <xacro:wamv_gps name="gps" x="-1.0" z="4.6" lat="44.09525149" lon="9.823435727" update_rate="20" />
-  <xacro:include filename="$(find mrc_examples)/urdf/cora_imu.xacro"/>
-  <xacro:cora_imu name="imu" y="-0.2" z="1.0" update_rate="100" />
-  <xacro:wamv_pinger name="pinger" frameId="cora/pinger" />
+  <xacro:wamv_camera name="front_left_camera"  x="-0.61" y="0.2"  z="4.7"
+  post_z_from="4.6" P="${radians(15)}" />
+  <xacro:wamv_camera name="front_right_camera" x="-0.61" y="-0.2" z="4.7"
+  post_z_from="4.6" P="${radians(15)}" />
+  <xacro:lidar name="front_lidar" type="16_beam" x="-0.595" z="5"
+  P="${radians(8)}" post_z_from="4.6"/>
+  <xacro:wamv_gps name="gps" x="-1.0" z="4.6"
+  	update_rate="20" />
+  <xacro:wamv_imu name="imu" y="-0.2" z="1.0" update_rate="100" />
  <gazebo>
       <plugin name="p3d_plugin_cora" filename="libgazebo_ros_p3d.so">
-        <bodyName>base_link</bodyName>
+        <bodyName>cora/base_link</bodyName>
         <frameName>map</frameName>
         <updateRate>10.0</updateRate>

Commit message: update for 2021

File: urdf/cora_p3d.xacro (robot description, xacro)
@@ -13,7 +13,11 @@
   <xacro:property name="namespace" value="$(arg namespace)" scope="global" />
   <!-- Thrusters -->
+  <!-- Thrusters mess this up - so this is hack - TODO Fix! -->
+  <xacro:arg name="root_namespace" default=""/>
+  <xacro:property name="root_namespace" value="$(arg root_namespace)" scope="global" />
   <xacro:arg name="thruster_namespace" default="thrusters/"/>
   <xacro:property name="thruster_namespace" value="$(arg thruster_namespace)" scope="global" />
-  <xacro:include filename="$(find cora_description)/urdf/thrusters.xacro" />
+  <!--<xacro:include filename="$(find cora_description)/urdf/thrusters.xacro" />-->
+  <xacro:include filename="$(find mrc_examples)/urdf/thrusters.xacro" />
   <!-- Decide if we lock the robot to the world -->
   <xacro:if value="$(arg locked)">

File: urdf/thrusters.xacro (robot description, xacro)
@@ -41,5 +41,5 @@
     <axis xyz="0 0 1"/>
     <origin rpy="0 0 0" xyz="-6.103 0.911 0.016"/>
-    <parent link="base_link"/>
+    <parent link="cora/base_link"/>
     <child link="left_engine_link"/>
     <limit lower="${-pi}" upper="${pi}" effort="10" velocity="10"/>
@@ -93,5 +93,5 @@
     <axis xyz="0 0 1"/>
     <origin rpy="0 0 0" xyz="-6.103 -0.911 0.016"/>
-    <parent link="base_link"/>
+    <parent link="cora/base_link"/>
     <child link="right_engine_link"/>
     <limit lower="${-pi}" upper="${pi}" effort="10" velocity="10"/>

Commit message: Working tf frames

File: urdf/cora_p3d.xacro (robot description, xacro)
@@ -1,51 +1,5 @@
 <?xml version="1.0"?>
 <robot xmlns:xacro="http://ros.org/wiki/xacro" name="cora">
-  <xacro:arg name="locked" default="false" />
-  <!-- Include macros for dynamics plugins -->
-  <xacro:include filename="$(find cora_description)/urdf/macros.xacro" />
-  <!-- Attach hydrodynamics plugin -->
-  <xacro:usv_dynamics_gazebo name="cora_dynamics_plugin" />
-  <!-- Robot mesh -->
-  <xacro:include filename="$(find cora_description)/urdf/cora.urdf.xacro" />
-  <!-- Note: this is only used for some sensors that do not correctly use the
-  robotNamespace parameter -->
-  <xacro:arg name="namespace" default="cora"/>
-  <xacro:property name="namespace" value="$(arg namespace)" scope="global" />
-  <!-- Thrusters -->
-  <!-- Thrusters mess this up - so this is hack - TODO Fix! -->
-  <xacro:arg name="root_namespace" default=""/>
-  <xacro:property name="root_namespace" value="$(arg root_namespace)" scope="global" />
-  <xacro:arg name="thruster_namespace" default="thrusters/"/>
-  <xacro:property name="thruster_namespace" value="$(arg thruster_namespace)" scope="global" />
-  <!--<xacro:include filename="$(find cora_description)/urdf/thrusters.xacro" />-->
-  <xacro:include filename="$(find mrc_examples)/urdf/thrusters.xacro" />
-  <!-- Decide if we lock the robot to the world -->
-  <xacro:if value="$(arg locked)">
-    <gazebo>
-      <link name="cora_external_link"/>
-      <joint name="cora_external_pivot_joint" type="universal">
-        <parent>cora::cora/base_link</parent>
-        <child>cora_external_link</child>
-        <axis>
-          <xyz>1 0 0</xyz>
-        </axis>
-        <axis2>
-          <xyz>0 1 0</xyz>
-        </axis2>
-      </joint>
-      <joint name="cora_external_riser" type="prismatic">
-        <parent>world</parent>
-        <child>cora_external_link</child>
-        <axis>
-          <limit>
-            <lower>-3</lower>
-            <upper>3</upper>
-          </limit>
-          <xyz>0 0 1</xyz>
-        </axis>
-      </joint>
-    </gazebo>
-  </xacro:if>
-  <!-- Sensors -->
+  <!-- Arguments and Parameters -->
   <xacro:arg name="camera_namespace" default="cameras/"/>
   <xacro:arg name="sensor_namespace" default="sensors/"/>
@@ -54,23 +8,56 @@
   <xacro:property name="sensor_namespace" value="$(arg sensor_namespace)" scope="global" />
   <xacro:property name="pinger_namespace" value="$(arg pinger_namespace)" scope="global" />
+  <!-- Note: this is only used for some sensors that do not correctly use the
+  robotNamespace parameter -->
+  <xacro:arg name="namespace" default="cora"/>
+  <xacro:property name="namespace" value="$(arg namespace)" scope="global" />
+  <!-- Thrusters mess this up - so this is hack - TODO Fix! -->
+  <xacro:arg name="root_namespace" default=""/>
+  <xacro:property name="root_namespace" value="$(arg root_namespace)" scope="global" />
+  <xacro:arg name="thruster_namespace" default="thrusters/"/>
+  <xacro:property name="thruster_namespace" value="$(arg thruster_namespace)" scope="global" />
+  <xacro:arg name="tf_prefix" default="cora1" />
+  <xacro:property name="tf_prefix" value="$(arg tf_prefix)" scope="global" />
+  <!-- Robot mesh -->
+  <xacro:include filename="$(find mrc_examples)/urdf/cora.urdf.xacro" />
+  <!-- Hydrodynamics plugin -->
+  <xacro:include filename="$(find mrc_examples)/urdf/cora_dynamics_plugin.xacro" />
+  <xacro:usv_dynamics_gazebo name="cora_dynamics_plugin" />
+  <!-- Thrusters -->
+  <xacro:include filename="$(find mrc_examples)/urdf/thrusters.xacro" />
+  <!-- P3D -->
+  <gazebo>
+    <plugin name="p3d_plugin_cora" filename="libgazebo_ros_p3d.so">
+      <bodyName>${tf_prefix}/cora/base_link</bodyName>
+      <frameName>map</frameName>
+      <updateRate>10.0</updateRate>
+      <topicName>cora/sensors/p3d</topicName>
+      <xyzOffset>0 0 0</xyzOffset>
+      <rpyOffset>0 0 0</rpyOffset>
+      <gaussianNoise>0</gaussianNoise>
+    </plugin>
+  </gazebo>
+  <!-- Lidar -->
+  <xacro:include filename="$(find mrc_examples)/urdf/cora_3d_lidar.xacro"/>
+  <xacro:cora_3d_lidar name="lidar"
+                           x="-0.595" y="0" z="5"
+                           R="0" P="0" Y="0"
+                           post_Y="0" post_z_from="4.6"
+                           vertical_lasers="16"/>
+  <!-- GPS
+  <xacro:include filename="$(find wamv_gazebo)/urdf/components/wamv_gps.xacro" />
+  <xacro:wamv_gps name="gps" x="-1.0" z="4.6"
+  		  update_rate="20" />
+  -->
+  <!-- IMU
+  <xacro:include filename="$(find wamv_gazebo)/urdf/components/wamv_imu.xacro" />
+  <xacro:wamv_imu name="imu" y="-0.2" z="1.0" update_rate="100" />
+  -->
+  <!-- Cameras
+  <xacro:include filename="$(find wamv_gazebo)/urdf/components/wamv_camera.xacro" /
   <xacro:wamv_camera name="front_left_camera"  x="-0.61" y="0.2"  z="4.7"
   post_z_from="4.6" P="${radians(15)}" />
   <xacro:wamv_camera name="front_right_camera" x="-0.61" y="-0.2" z="4.7"
   post_z_from="4.6" P="${radians(15)}" />
-  <xacro:lidar name="front_lidar" type="16_beam" x="-0.595" z="5"
-  P="${radians(8)}" post_z_from="4.6"/>
-  <xacro:wamv_gps name="gps" x="-1.0" z="4.6"
-  	update_rate="20" />
-  <xacro:wamv_imu name="imu" y="-0.2" z="1.0" update_rate="100" />
- <gazebo>
-      <plugin name="p3d_plugin_cora" filename="libgazebo_ros_p3d.so">
-        <bodyName>cora/base_link</bodyName>
-        <frameName>map</frameName>
-        <updateRate>10.0</updateRate>
-        <topicName>cora/sensors/p3d</topicName>
-        <xyzOffset>0 0 0</xyzOffset>
-        <rpyOffset>0 0 0</rpyOffset>
-        <gaussianNoise>0</gaussianNoise>
-      </plugin>
-</gazebo>
+  -->
 </robot>

File: urdf/thrusters.xacro (robot description, xacro)
@@ -2,5 +2,5 @@
 <robot xmlns:xacro="http://ros.org/wiki/xacro">
   <!-- Dummy link, which usv_gazebo_thrust_plugin looks for -->
-  <link name="left_engine_link">
+  <link name="${tf_prefix}/${namespace}/left_engine_link">
     <inertial>
       <mass value="0.1"/>
@@ -9,5 +9,5 @@
   </link>
   <!-- No additional collision, since propeller is inside robot body -->
-  <link name="left_propeller_link">
+  <link name="${tf_prefix}/${namespace}/left_propeller_link">
     <visual>
       <geometry>
@@ -38,21 +38,21 @@
   </link>
   <!-- Dummy joint, which usv_gazebo_thrust_plugin looks for -->
-  <joint name="left_chasis_engine_joint" type="revolute">
+  <joint name="${tf_prefix}/${namespace}/left_chasis_engine_joint" type="revolute">
     <axis xyz="0 0 1"/>
     <origin rpy="0 0 0" xyz="-6.103 0.911 0.016"/>
-    <parent link="cora/base_link"/>
-    <child link="left_engine_link"/>
+    <parent link="${tf_prefix}/${namespace}/base_link"/>
+    <child link="${tf_prefix}/${namespace}/left_engine_link"/>
     <limit lower="${-pi}" upper="${pi}" effort="10" velocity="10"/>
   </joint>
-  <joint name="left_engine_propeller_joint" type="continuous">
+  <joint name="${tf_prefix}/${namespace}/left_engine_propeller_joint" type="continuous">
     <axis rpy="0 0 0" xyz="1 0 0"/>
     <origin xyz="0 0 0" rpy="0 0 0"/>
-    <parent link="left_engine_link"/>
-    <child link="left_propeller_link"/>
+    <parent link="${tf_prefix}/${namespace}/left_engine_link"/>
+    <child link="${tf_prefix}/${namespace}/left_propeller_link"/>
     <limit effort="100" velocity="100" />
     <dynamics friction="0.05" damping="0.05" />
   </joint>
   <!-- Dummy link, which usv_gazebo_thrust_plugin looks for -->
-  <link name="right_engine_link">
+  <link name="${tf_prefix}/${namespace}/right_engine_link">
     <inertial>
       <mass value="0.1"/>
@@ -61,5 +61,5 @@
   </link>
   <!-- No additional collision, since propeller is inside robot body -->
-  <link name="right_propeller_link">
+  <link name="${tf_prefix}/${namespace}/right_propeller_link">
     <visual>
       <geometry>
@@ -90,16 +90,16 @@
   </link>
   <!-- Dummy joint, which usv_gazebo_thrust_plugin looks for -->
-  <joint name="right_chasis_engine_joint" type="revolute">
+  <joint name="${tf_prefix}/${namespace}/right_chasis_engine_joint" type="revolute">
     <axis xyz="0 0 1"/>
     <origin rpy="0 0 0" xyz="-6.103 -0.911 0.016"/>
-    <parent link="cora/base_link"/>
-    <child link="right_engine_link"/>
+    <parent link="${tf_prefix}/${namespace}/base_link"/>
+    <child link="${tf_prefix}/${namespace}/right_engine_link"/>
     <limit lower="${-pi}" upper="${pi}" effort="10" velocity="10"/>
   </joint>
-  <joint name="right_engine_propeller_joint" type="continuous">
+  <joint name="${tf_prefix}/${namespace}/right_engine_propeller_joint" type="continuous">
     <axis rpy="0 0 0" xyz="1 0 0"/>
     <origin xyz="0 0 0" rpy="0 0 0"/>
-    <parent link="right_engine_link"/>
-    <child link="right_propeller_link"/>
+    <parent link="${tf_prefix}/${namespace}/right_engine_link"/>
+    <child link="${tf_prefix}/${namespace}/right_propeller_link"/>
     <limit effort="100" velocity="100" />
     <dynamics friction="0.05" damping="0.05" />
@@ -108,9 +108,36 @@
     <plugin name="cora_gazebo_thrust" filename="libusv_gazebo_thrust_plugin.so">
       <cmdTimeout>1.0</cmdTimeout>
-      <robotNamespace>${root_namespace}/${namespace}</robotNamespace>
-      <xacro:include filename="$(find cora_description)/urdf/cora_thruster_config.xacro" />
-      <!-- Angle must be disabled for VORC -->
-      <xacro:cora_thruster_config name="left" />
-      <xacro:cora_thruster_config name="right" />
+      <!-- Left -->
+      <thruster>
+	<!-- Required Parameters -->
+	<linkName>${tf_prefix}/${namespace}/left_propeller_link</linkName>
+	<propJointName>${tf_prefix}/${namespace}/left_engine_propeller_joint</propJointName>
+	<engineJointName>${tf_prefix}/${namespace}/left_chasis_engine_joint</engineJointName>
+	<cmdTopic>${tf_prefix}/${namespace}/left_thrust_cmd</cmdTopic>
+	<angleTopic>${tf_prefix}/${namespace}/left_thrust_angle</angleTopic>
+	<enableAngle>false</enableAngle>
+	<!-- Optional Parameters -->
+	<mappingType>0</mappingType>
+	<maxCmd>1.0</maxCmd>
+	<maxForceFwd>120000.0</maxForceFwd>
+	<maxForceRev>-50000.0</maxForceRev>
+	<maxAngle>${pi/2}</maxAngle>
+      </thruster>
+      <!-- Right -->
+      <thruster>
+	<!-- Required Parameters -->
+	<linkName>${tf_prefix}/${namespace}/right_propeller_link</linkName>
+	<propJointName>${tf_prefix}/${namespace}/right_engine_propeller_joint</propJointName>
+	<engineJointName>${tf_prefix}/${namespace}/right_chasis_engine_joint</engineJointName>
+	<cmdTopic>${tf_prefix}/${namespace}/right_thrust_cmd</cmdTopic>
+	<angleTopic>${tf_prefix}/${namespace}/right_thrust_angle</angleTopic>
+	<enableAngle>false</enableAngle>
+	<!-- Optional Parameters -->
+	<mappingType>0</mappingType>
+	<maxCmd>1.0</maxCmd>
+	<maxForceFwd>120000.0</maxForceFwd>
+	<maxForceRev>-50000.0</maxForceRev>
+	<maxAngle>${pi/2}</maxAngle>
+      </thruster>
     </plugin>
   </gazebo>
